File: docs/usdx_kicad/usdx_kicad.kicad_pcb (KiCad board)
At the start: 2 copper layers, 153 x 134.5 mm, 73 parts, among them J10 Speaker, J11 Power Connector, J12 +12V, J13 MCP23017, J3 SSD1309, J4 PWR SWR meter, J5 W5500, J6 ROT_MENU, J7 ROT_FREQ, J8 Button Right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

Commit message: PCB version 1.1
Parts:
- removed ? (x2): , 
- removed R3, R4, R5, R6: 100, Resistor_THT:R_Axial_DIN0207_L6.3mm_D2.5mm_P7.62mm_Horizontal
- removed REF**, RX: MountingHole_2.7mm, MountingHole:MountingHole_2.7mm
- removed RX J1: RX input, Connector_Coaxial:SMA_Molex_73251-1153_EdgeMount_Horizontal
- removed TX J2: TX, Connector_Coaxial:SMA_Molex_73251-1153_EdgeMount_Horizontal
- added C30: 10u, Capacitor_THT:C_Disc_D5.0mm_W2.5mm_P5.00mm, F.Cu at (131.5, 135.5)
- added C31: 10u, Capacitor_THT:C_Disc_D5.0mm_W2.5mm_P5.00mm, F.Cu at (131.5, 139.5)
- added C32: 10u, Capacitor_THT:C_Disc_D5.0mm_W2.5mm_P5.00mm, F.Cu at (131.5, 127.5)
- added C33: 10u, Capacitor_THT:C_Disc_D5.0mm_W2.5mm_P5.00mm, F.Cu at (131.5, 131.5)
- added R13: 10K, Resistor_THT:R_Axial_DIN0207_L6.3mm_D2.5mm_P7.62mm_Horizontal, F.Cu at (136.0, 143.1)
- added R14: 10K, Resistor_THT:R_Axial_DIN0207_L6.3mm_D2.5mm_P7.62mm_Horizontal, F.Cu at (139.5, 143.1)
- added U3: RX Input, myFootprintLibrary:SMA connector, F.Cu at (76.3, 150.5)
- added U4: TX Out, myFootprintLibrary:SMA connector, F.Cu at (76.3, 114.0)
- C5, C6, C7, C8: value 1n -> 220n
- U1: footprint Espressif:ESP32-S3-DevKitC -> myFootprintLibrary:ESP32-S3-DevKitC-Mine
- moved R10 0.91 mm to (141.7, 64.6)
- moved R11 0.91 mm to (138.2, 64.6)
- renumbered MAX98357 to MAX98357_board1, PCM1808 to PCM1, SI5351 to SI5351_board1, LM4562 to U2
Routing:
- net GND: track 82.7 -> 0.00 mm, vias 35 -> 49
- net Net-(T1-SB): track 20.4 -> 53.0 mm
- net Net-(U2B--): track 22.6 -> 36.6 mm
- net Net-(T1-AB): track 19.3 -> 29.1 mm
- net Net-(FST3253-2B1): track 46.4 -> 39.6 mm
- net Net-(U2A--): track 29.5 -> 33.9 mm
- net /ROT_FREQ_DT: track 178.9 -> 183.0 mm
- net Net-(FST3253-2B4): track 32.0 -> 28.8 mm
- net Net-(FST3253-2B3): track 28.5 -> 25.6 mm
- net Net-(FST3253-2B2): track 26.7 -> 23.8 mm
- net Net-(SI5351_board1-CLK2): track 31.2 -> 33.9 mm
- net /ROT_MENU_DT: track 110.9 -> 113.6 mm
- net /ROT_MENU_SW: track 115.0 -> 117.7 mm
- net Net-(U2A-+): track 45.9 -> 48.4 mm
- net /ROT_MENU_CLK: track 106.7 -> 109.1 mm
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Other:
- board text added: "+19V"
- board text added: "Button Left"
- board text added: "Button Right"
- board text added: "FT8-ESP32 V1.1 by Guido - IW5ALZ 21/06/2026"
- board text added: "MCP23017"
- board text added: "PWR SWR METER"
- board text added: "ROT Freq"
- board text added: "ROT Menu"
- board text added: "RX IN"
- board text added: "SSD1309"
- board text added: "Speaker"
- board text added: "TX OUT"
- board text added: "W5500"

Commit message: set \r\n in all printf
Other:
- board text added: "+19Vr"
- board text added: "Button Leftr"
- board text added: "Button Rightr"
- board text added: "FT8-ESP32 V1.1r by Guido - IW5ALZr 21/06/2026"
- board text added: "MCP23017r"
- board text added: "PWR SWRr METER"
- board text added: "ROT Freqr"
- board text added: "ROT Menur r"
- board text added: "RX INr"
- board text added: "TX OUTr"
- board text added: "W5500r"
- board text removed: "+19V"
- board text removed: "Button Left"
- board text removed: "Button Right"
- board text removed: "FT8-ESP32 V1.1 by Guido - IW5ALZ 21/06/2026"
- board text removed: "MCP23017"
- board text removed: "PWR SWR METER"
- board text removed: "ROT Freq"
- board text removed: "ROT Menu"
- board text removed: "RX IN"
- board text removed: "TX OUT"
- board text removed: "W5500"
Changed lines of the file:
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@@
 		(layer "Edge.Cuts")
 	)
-	(gr_text "TX OUT\n"
+	(gr_text "TX OUT\r\n"
 		(at 80 114.000001 0)
 		(layer "F.SilkS")
@@
 		)
 	)
-	(gr_text "W5500\n"
+	(gr_text "W5500\r\n"
 		(at 80.38 48 0)
 		(layer "F.SilkS")
@@
 		)
 	)
-	(gr_text "RX IN\n"
+	(gr_text "RX IN\r\n"
 		(at 80.5 150.5 0)
 		(layer "F.SilkS")
@@
 		)
 	)
-	(gr_text "PWR SWR\nMETER"
+	(gr_text "PWR SWR\r\nMETER"
 		(at 81 74 0)
 		(layer "F.SilkS")
@@
 		)
 	)
-	(gr_text "MCP23017\n"
+	(gr_text "MCP23017\r\n"
 		(at 81 81 0)
 		(layer "F.SilkS")
@@
 		)
 	)
-	(gr_text "Button Right\n"
+	(gr_text "Button Right\r\n"
 		(at 212 49 0)
 		(layer "F.SilkS")
@@
 		)
 	)
-	(gr_text "Button Left\n"
+	(gr_text "Button Left\r\n"
 		(at 213.5 137.5 0)
 		(layer "F.SilkS")
@@
 		)
 	)
-	(gr_text "ROT Freq\n"
+	(gr_text "ROT Freq\r\n"
 		(at 214.5 62 0)
 		(layer "F.SilkS")
@@
 		)
 	)
-	(gr_text "ROT Menu\n\n"
+	(gr_text "ROT Menu\r\n\r\n"
 		(at 214.5 135.5 0)
 		(layer "F.SilkS")
@@
 		)
 	)
-	(gr_text "+19V\n"
+	(gr_text "+19V\r\n"
 		(at 76.5 36 0)
 		(layer "F.SilkS")
@@
 		)
 	)
-	(gr_text "FT8-ESP32 V1.1\nby Guido - IW5ALZ\n21/06/2026"
+	(gr_text "FT8-ESP32 V1.1\r\nby Guido - IW5ALZ\r\n21/06/2026"
 		(at 194 162.5 0)
 		(layer "F.SilkS")
